File: rc2014_de10_adapter.sch (KiCad schematic (older format))
At the start: 19 parts, among them J1 Z80 Bus, J2 Pro Bus, J3 Conn_02x20_Odd_Even, J4 M3 Mounting Hole, J5 Conn_01x10_Male, J6 Conn_01x08_Male, U1 SN74LVC245A, U10 MAX40200AUK, U2 SN74LVC245A, U3 SN74LVC245A, U4 SN74LVC245A, U5 AZ1117-3.3, U6 SN74LVC245A, U7 MAX40200AUK, U8 MAX40200AUK, U9 MAX40200AUK

Commit message: reorganized schematic
Parts:
- removed U7, U8: MAX40200AUK, Package_TO_SOT_SMD:SOT-23-5, symbol Analog_Switch:MAX40200AUK
- added C10, C5, C6, C9: 1uF, Capacitor_SMD:C_0805_2012Metric_Pad1.15x1.40mm_HandSolder, symbol Device:C
- added C11, C4, C7, C8: 100nF, Capacitor_SMD:C_0805_2012Metric_Pad1.15x1.40mm_HandSolder, symbol Device:C
- added U10, U9: MAX40200AUK, Package_TO_SOT_SMD:SOT-23-5, symbol Analog_Switch:MAX40200AUK
- U1, U2, U3: symbol dk_Logic-Buffers-Drivers-Receivers-Transceivers:SN74LVC245A -> rc2014_de10_adapter-rescue:SN74LVC245A-dk_Logic-Buffers-Drivers-Receivers-Transceivers
- U4: renamed from U6; symbol dk_Logic-Buffers-Drivers-Receivers-Transceivers:SN74LVC245A -> rc2014_de10_adapter-rescue:SN74LVC245A-dk_Logic-Buffers-Drivers-Receivers-Transceivers
- U5: renamed from U4; symbol dk_Logic-Buffers-Drivers-Receivers-Transceivers:SN74LVC245A -> rc2014_de10_adapter-rescue:SN74LVC245A-dk_Logic-Buffers-Drivers-Receivers-Transceivers
- renumbered J3 to J1, J5 to J2, J6 to J3, J1 to J5, J2 to J6, U5 to U6, U9 to U7, U10 to U8
Connections:
- net 5V is gone; now on net +5V: C1.2, C2.1, J5.18 (Pin_18), J6.2 (Pin_2), U6.3 (VI), U7.1 (VDD), U7.3 (EN)
- net ~RESET2 is gone; now on net PAGE: J6.4 (Pin_4)
- net +3V3: now also U1.1 (DIR), U2.1 (DIR), U3.1 (DIR), C10.2, C11.2, C8.2, C9.2, U10.5 (OUT), U9.5 (OUT)
- net +5V: now also C4.2, C5.2, C6.2, C7.2
- net 3V3: now also U9.1 (VDD), U9.3 (EN)
- net 3V3F: now also U10.1 (VDD), U10.3 (EN)
- net GND: now also C10.1, C11.1, C4.1, C5.1, C6.1, C7.1, C8.1, C9.1, U10.2 (GND), U9.2 (GND); no longer U1.1 (DIR), U2.1 (DIR), U3.1 (DIR), U5.1 (DIR)
- net Tx: now reaches J5.35 (Pin_35)
- net Tx: now also U3.9 (A8)
- net Rx: now reaches J5.36 (Pin_36)
- net Rx: now also U4.9 (A8)
- net PAGEF: now reaches J2.9 (Pin_9)
- net PAGEF: now also U4.12 (B7)
- net RxF: now reaches J3.1 (Pin_1)
- net RxF: now also U4.11 (B8)
- net TxF: now reaches J3.2 (Pin_2)
- net TxF: now also U3.11 (B8)
- net DIR: now reaches J3.8 (Pin_8)
- net DIR: now also U5.1 (DIR)
- net PAGE: now reaches U4.8 (A7)
- no-connect marks 30 -> 17
Other:
- moved on the sheet: C1, C2, C3, J4, U1, U2, U3, U4, U5, U6, U7, U8
